File: Hardware/projet_elec_midi/projet_elec_midi.kicad_pcb (KiCad board)
At the start: 2 copper layers, 76 parts, among them J1 Conn_01x02, U1 STM32G431KBTx, U2 MCP73811T-420I-OT, U3 USBLC6-2SC6, U4 74HC4051, U5 74HC4051, U6 74HC4051, U7 74HC4051

Commit message: Kicad schematic terminée
Parts:
- removed RV28: B100k, Potentiometer_THT:Potentiometer_Bourns_PTA3043_Single_Slide
- added C1: 4.7u, Capacitor_SMD:C_0603_1608Metric, F.Cu at (225.1, 71.7)
- added C2: 1u, Capacitor_SMD:C_0603_1608Metric, F.Cu at (239.7, 107.4)
- added C3: 100n, Capacitor_SMD:C_0603_1608Metric, F.Cu at (225.1, 74.2)
- added C4: 100n, Capacitor_SMD:C_0603_1608Metric, F.Cu at (225.1, 76.8)
- added C44: 10n, Capacitor_SMD:C_0603_1608Metric, F.Cu at (225.1, 84.3)
- added C45: 1u, Capacitor_SMD:C_0603_1608Metric_Pad1.08x0.95mm_HandSolder, F.Cu at (237.0, 97.4)
- added C46: 1u, Capacitor_SMD:C_0603_1608Metric_Pad1.08x0.95mm_HandSolder, F.Cu at (237.0, 99.9)
- added C5: 1u, Capacitor_SMD:C_0603_1608Metric, F.Cu at (239.7, 109.9)
- added C6: 100n, Capacitor_SMD:C_0603_1608Metric, F.Cu at (225.1, 79.3)
- added C7: 1u, Capacitor_SMD:C_0603_1608Metric, F.Cu at (225.1, 81.8)
- added H1: MountingHole_Pad, MountingHole:MountingHole_3.2mm_M3_Pad_Via, F.Cu at (204.9, 74.5)
- added H2: MountingHole_Pad, MountingHole:MountingHole_3.2mm_M3_Pad_Via, F.Cu at (204.9, 82.4)
- added H3: MountingHole_Pad, MountingHole:MountingHole_3.2mm_M3_Pad_Via, F.Cu at (204.9, 90.3)
- added H4: MountingHole_Pad, MountingHole:MountingHole_3.2mm_M3_Pad_Via, F.Cu at (204.9, 98.3)
- added J3: Conn_02x07_Odd_Even, Connector_PinHeader_1.27mm:PinHeader_2x07_P1.27mm_Vertical_SMD, F.Cu at (270.3, 80.2)
- added J4: MIDI, Connector_Audio:Jack_3.5mm_CUI_SJ-3523-SMT_Horizontal, F.Cu at (215.0, 80.0)
- added J5: USB_C_Receptacle_USB2.0_16P, Connector_USB:USB_C_Receptacle_GCT_USB4105-xx-A_16P_TopMnt_Horizontal, F.Cu at (229.0, 101.4)
- added JP1: SolderJumper_3_Bridged12, Jumper:SolderJumper-3_P1.3mm_Bridged12_RoundedPad1.0x1.5mm, F.Cu at (211.7, 91.3)
- added JP2: SolderJumper_3_Bridged12, Jumper:SolderJumper-3_P1.3mm_Bridged12_RoundedPad1.0x1.5mm, F.Cu at (211.7, 95.1)
- added L1: 39n, Inductor_SMD:L_0805_2012Metric, F.Cu at (239.1, 71.8)
- added R1: 5.1k, Resistor_SMD:R_0603_1608Metric, F.Cu at (239.7, 112.4)
- added R2: 5.1k, Resistor_SMD:R_0603_1608Metric, F.Cu at (239.7, 114.9)
- added R3: 100k, Resistor_SMD:R_0603_1608Metric, F.Cu at (225.1, 86.8)
- added R4: 10R, Resistor_SMD:R_0805_2012Metric, F.Cu at (216.7, 91.0)
- added R5: 33R, Resistor_SMD:R_0805_2012Metric, F.Cu at (216.7, 94.0)
- added RVE: B10K, Potentiometer_THT:Potentiometer_Bourns_PTA3043_Single_Slide, F.Cu at (110.0, 130.0)
- added U8: MCP1802x-xx02xOT, Package_TO_SOT_SMD:SOT-23-5, F.Cu at (235.2, 117.2)
- J1: value Conn_01x02 -> BATTERY
- RV25, RV26, RV27, RV29, RV30, RV31, RV32: value B100k -> B10K
- moved C26 239.8 mm to (281.7, 100.5)
- moved C27 239.8 mm to (281.7, 103.0)
- moved C28 239.8 mm to (281.7, 105.5)
- moved C29 239.8 mm to (281.7, 108.1)
- moved C30 239.8 mm to (281.7, 110.6)
- moved C31 239.8 mm to (281.7, 113.1)
- moved C32 239.8 mm to (281.7, 115.6)
- moved C33 239.8 mm to (281.7, 118.1)
- moved C34 239.8 mm to (281.7, 120.6)
- moved U2 187.1 mm to (235.2, 108.3)
- moved U3 187.1 mm to (235.2, 112.8)
- moved J1 185.1 mm to (226.6, 109.5)
- moved U1 184.7 mm to (232.8, 88.4)
- moved C13 178.7 mm to (281.7, 60.8)
- moved C14 178.7 mm to (281.7, 63.3)
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Connections:
- net Net-(J1-Pin_1) renamed +BATT
- net voie 0 renamed /voie0
- net voie 1 renamed /voie1
- net voie 2 renamed /voie2
- net voie 3 renamed /voie3
- RV25 pad MP: (no net) -> GND
- RV26 pad MP: (no net) -> GND
- RV27 pad MP: (no net) -> GND
- RV29 pad MP: (no net) -> GND
- RV30 pad MP: (no net) -> GND
- RV31 pad MP: (no net) -> GND
- RV32 pad MP: (no net) -> GND
- U1 pad 10: sel 0 -> /sel1
- U1 pad 11: sel 1 -> /sel2
- U1 pad 12: sel 2 -> unconnected-(U1-PA7-Pad12)
- U1 pad 19: unconnected-(U1-PA9-Pad19) -> /STM32/USART1_TX
- U1 pad 20: unconnected-(U1-PA10-Pad20) -> /STM32/USART1_RX
- U1 pad 21: unconnected-(U1-PA11-Pad21) -> /D-
- U1 pad 22: unconnected-(U1-PA12-Pad22) -> /D+
- U1 pad 23: unconnected-(U1-PA13-Pad23) -> /STM32/SYS_SWDIO
- U1 pad 24: unconnected-(U1-PA14-Pad24) -> /STM32/SYS_SWCLK
- U1 pad 26: unconnected-(U1-PB3-Pad26) -> /MIDI_TX
- U1 pad 31: unconnected-(U1-PB8-Pad31) -> /STM32/BOOT0
- U1 pad 4: unconnected-(U1-PG10-Pad4) -> /STM32/NRST
- U1 pad 9: unconnected-(U1-PA4-Pad9) -> /sel0
- U2 pad 1: +5V -> VBUS
- U2 pad 4: +5V -> VBUS
- U2 pad 5: +5V -> VBUS
- U3 pad 3: D+ -> /D+
- U3 pad 4: D- -> /D-
- U4 pad 10: sel 1 -> /sel1
- U4 pad 11: sel 0 -> /sel0
- U4 pad 9: sel 2 -> /sel2
- U5 pad 10: sel 1 -> /sel1
- U5 pad 11: sel 0 -> /sel0
- U5 pad 9: sel 2 -> /sel2
- U6 pad 10: sel 1 -> /sel1
- U6 pad 11: sel 0 -> /sel0
- U6 pad 9: sel 2 -> /sel2
- U7 pad 10: sel 1 -> /sel1
- U7 pad 11: sel 0 -> /sel0
- U7 pad 9: sel 2 -> /sel2

Commit message: Kicad début du routage
Parts:
- moved J3 268.4 mm to (25.1, 189.3)
- moved C27 264.6 mm to (18.8, 73.4)
- moved C28 243.7 mm to (40.0, 74.4)
- moved H1 227.3 mm to (15.0, 199.4)
- moved C29 225.1 mm to (59.0, 75.2), turned to -90 degrees
- moved J5 215.6 mm to (26.8, 26.7), turned to 180 degrees
- moved C30 205.9 mm to (79.0, 74.4)
- moved HE 205.3 mm to (15.0, 12.4)
- moved C13 190.4 mm to (99.0, 114.4)
- moved C31 186.9 mm to (99.0, 73.4)
- moved C14 170.5 mm to (119.0, 114.4)
- moved C32 167.8 mm to (119.0, 74.4)
- moved RV17 156.6 mm to (23.5, 71.4)
- moved RV9 156.1 mm to (23.5, 91.4)
- moved C18 153.2 mm to (19.2, 96.4), turned to 180 degrees
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- renumbered H3 to HE, RVE to RV28
Routing:
- added copper zone on B.Cu, net GND
- added copper zone on F.Cu, net GND

Commit message: Routage en double face
Parts:
- C1, C17, C2, C26, C3, C35, C4, C44, C45, C46, C5, C6, C7, C8, J1, J3, J4, J5, JP1, JP2, L1, R1, R2, R3, R4, R5, U1, U2, U3, U4, U5, U6, U7, U8: moved to B.Cu
- moved C35 256.9 mm to (23.0, 149.6), turned to 90 degrees
- moved C43 234.8 mm to (28.7, 128.5), turned to 180 degrees
- moved C42 217.8 mm to (47.7, 128.0), turned to 180 degrees
- moved C46 208.1 mm to (49.4, 41.1), turned to 180 degrees
- moved C45 204.3 mm to (49.3, 47.2), turned to 180 degrees
- moved U8 203.3 mm to (49.3, 44.2), turned to 90 degrees
- moved R2 201.1 mm to (71.0, 46.7)
- moved C5 198.5 mm to (53.5, 52.1), turned to -90 degrees
- moved C17 196.2 mm to (47.7, 98.2), turned to 180 degrees
- moved C2 191.9 mm to (59.5, 52.6), turned to -90 degrees
- moved U2 190.8 mm to (56.4, 52.6)
- moved R1 189.3 mm to (81.6, 46.8), turned to 90 degrees
- moved U1 188.2 mm to (88.0, 51.0), turned to 180 degrees
- moved C8 186.9 mm to (24.2, 120.3), turned to 180 degrees
- moved U3 175.0 mm to (77.0, 46.9), turned to 90 degrees
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- renumbered HE to H3
Connections:
- U3 pad 1: Net-(J5-D+-PadA6) -> /D+
- U3 pad 3: /D+ -> /D-
- U3 pad 4: /D- -> Net-(J5-D--PadA7)
- U3 pad 6: Net-(J5-D--PadA7) -> Net-(J5-D+-PadA6)
Routing:
- net VBUS: track 0.00 -> 15.1 mm, vias 0 -> 2
- net GND: track 0.00 -> 11.9 mm, vias 0 -> 8
- net /D-: track 0.00 -> 9.84 mm
- net +BATT: track 0.00 -> 7.63 mm
- net /D+: track 0.00 -> 7.26 mm
- net Net-(J5-D+-PadA6): track 0.00 -> 5.33 mm
- net Net-(J5-D--PadA7): track 0.00 -> 4.28 mm
- net +3.3V: track 0.00 -> 3.74 mm
Other:
- board outline added: 168 x 148 mm
