File: Hardware/projet_elec_midi/projet_elec_midi.kicad_sch (KiCad schematic)
At the start: 21 parts, among them J1 Conn_01x02, J2 USB_C_Receptacle_USB2.0, J3 Conn_02x07_Odd_Even, U1 STM32G431KBTx, U2 MCP73811T-420I-OT, U3 USBLC6-2SC6

Commit message: Kicad schematic terminée
Parts:
- removed C1: 4.7u, symbol Device:C_Small
- removed C2, C5, C6: 1u, symbol Device:C_Small
- removed C3, C4: 100n, symbol Device:C_Small
- removed C44: 100n, Capacitor_SMD:C_0603_1608Metric_Pad1.08x0.95mm_HandSolder, symbol Device:C_Small
- removed C7: 10n, symbol Device:C_Small
- removed H1, H2, H3, H4: MountingHole, MountingHole:MountingHole_3.2mm_M3_DIN965_Pad, symbol Mechanical:MountingHole
- removed J1: Conn_01x02, Connector_JST:JST_XH_S2B-XH-A_1x02_P2.50mm_Horizontal, symbol Connector_Generic:Conn_01x02
- removed J2: USB_C_Receptacle_USB2.0, symbol Connector:USB_C_Receptacle_USB2.0
- removed J3: Conn_02x07_Odd_Even, Connector_PinHeader_1.27mm:PinHeader_2x08_P1.27mm_Vertical_SMD, symbol Connector_Generic:Conn_02x07_Odd_Even
- removed L1: 39n, symbol Device:L
- removed R1, R2: 5.1k, symbol Device:R_Small
- removed U1: STM32G431KBTx, Package_QFP:LQFP-32_7x7mm_P0.8mm, symbol MCU_ST_STM32G4:STM32G431KBTx
- removed U2: MCP73811T-420I-OT, Package_TO_SOT_SMD:SOT-23-5, symbol Battery_Management:MCP73811T-420I-OT
- removed U3: USBLC6-2SC6, Package_TO_SOT_SMD:SOT-23-6, symbol Power_Protection:USBLC6-2SC6
- added H1, H2, H3, H4: MountingHole_Pad, MountingHole:MountingHole_3.2mm_M3_Pad_Via, symbol Mechanical:MountingHole_Pad
- added J4: MIDI, Connector_Audio:Jack_3.5mm_CUI_SJ-3523-SMT_Horizontal, symbol Connector_Audio:AudioJack3
- added JP1, JP2: SolderJumper_3_Bridged12, Jumper:SolderJumper-3_P1.3mm_Bridged12_RoundedPad1.0x1.5mm, symbol Jumper:SolderJumper_3_Bridged12
- added R4: 10R, Resistor_SMD:R_0805_2012Metric, symbol Device:R_Small
- added R5: 33R, Resistor_SMD:R_0805_2012Metric, symbol Device:R_Small
Connections:
- net +3.3V: now also R5.1
- net GND: now also H1.1, H2.1, H3.1, H4.1, J4.S
- new net JACK_R: J4.R, JP2.2 (C)
- new net JACK_T: J4.T, JP1.2 (C)
- new net MIDI_TX: R4.1
- new net SINK: JP1.1 (A), JP2.3 (B), R4.2
- new net SOURCE: JP1.3 (B), JP2.1 (A), R5.2
- no-connect marks 10 -> 0
Other:
- added sheet Alimentation (alimentation.kicad_sch)
- added sheet STM32 (stm32.kicad_sch)
- note added: "Connecteur MIDI"
- note added: "Potentiomètres"
- note removed: "BATTERIE BMS"
- note removed: "Connecteur SWD de programmation du microcontrôleur"
- note removed: "On route ce composant au plus proche du connecteur USB"
- note removed: "PORT USB MIDI + RECHARGE"
- note removed: "STM32"
