File: Hardware/kicad new/projet_elec_midi.kicad_pcb (KiCad board)
At the start: 2 copper layers, 168 x 148 mm, 102 parts, among them J1 BATTERY, J3 Conn_02x07_Odd_Even, J4 MIDI, J5 USB_C_Receptacle_USB2.0_16P, U1 STM32G431KBTx, U2 MCP73811T-420I-OT, U3 USBLC6-2SC6, U4 74HC4051, U5 74HC4051, U6 74HC4051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

Commit message: Routage de la carte fini
Parts:
- moved C3 18.9 mm to (95.1, 47.1), turned to 0 degrees
- moved C44 13.6 mm to (86.7, 57.1), turned to 0 degrees
- moved C17 10.9 mm to (42.4, 88.7), turned to 0 degrees
- moved R4 10.4 mm to (136.8, 45.3), turned to 90 degrees
- moved R3 10.3 mm to (92.7, 55.9), turned to -90 degrees
- moved C34 7.66 mm to (172.1, 74.1)
- moved L1 7.21 mm to (80.9, 57.1), turned to 0 degrees
- moved C7 6.75 mm to (83.5, 56.3)
- moved R2 4.55 mm to (70.8, 42.2), turned to -90 degrees
- moved C8 4.06 mm to (25.6, 116.5)
- moved C4 3.70 mm to (94.2, 49.8)
- moved C18 3.45 mm to (30.2, 94.0)
- moved C10 3.31 mm to (52.1, 114.2)
- moved C6 2.84 mm to (81.9, 54.6), turned to -90 degrees
- moved C16 2.71 mm to (172.1, 114.3)
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Routing:
- net GND: track 56.5 -> 30.3 mm, vias 111 -> 108
- net +3.3V: track 835.4 -> 818.0 mm, vias 18 -> 8
- net +3.3VA: track 21.8 -> 6.05 mm, vias 2 -> 0
- net /MIDI_TX: track 57.7 -> 69.6 mm
- net /STM32/BOOT0: track 22.0 -> 10.5 mm
- net /potentiometer circular2/POT7: track 141.6 -> 131.4 mm, vias 2 -> 0
- net /SINK: track 23.2 -> 13.3 mm
- net /voie3: track 161.5 -> 170.7 mm, vias 3 -> 2
- net Net-(J5-CC1): track 12.8 -> 6.18 mm, vias 2 -> 0
- net /STM32/NRST: track 22.7 -> 18.9 mm
- net /voie2: track 72.7 -> 69.1 mm
- net +BATT: track 130.6 -> 127.3 mm, vias 3 -> 0
- net /potentiometer circular/POT4: track 82.1 -> 85.3 mm, vias 1 -> 0
- net /potentiometer circular1/POT0: track 14.0 -> 11.1 mm, vias 1 -> 0
- net /sel2: track 188.9 -> 186.3 mm, vias 8 -> 6
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